Commit message: 实现手柄控制接口

File: src/rm_engineering_robot_description/urdf/rm_engineering_robot.urdf (robot description, URDF)
Before this commit: robot rm_engineering_robot, 9 links, 8 joints
Links:
- link base_link: geometry collision box size=0.1 0.1 0.1; visual mesh filename=package://rm_engineering_robot_description/meshes/base_link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
