Commit message: 修改urdf

File: src/rm_engineering_robot_description/urdf/rm_engineering_robot.urdf (robot description, URDF)
Before this commit: robot rm_engineering_robot, 9 links, 8 joints
Links:
- added link zed_camera_link
Joints:
- added joint link3_to_zed_camera_link: type fixed, parent link5, child zed_camera_link, origin xyz=0.10 0.00 0.05 rpy=0.00 0.00 0.00

Commit message: 在foundationpose_bridge包添加mesh可视化，修改相机的URDF描述

File: src/rm_engineering_robot_description/urdf/rm_engineering_robot.urdf (robot description, URDF)
Before this commit: robot rm_engineering_robot, 10 links, 9 joints
Joints:
- joint link3_to_zed_camera_link: origin xyz=0.10 0.00 0.05 rpy=0.00 0.00 0.00 -> xyz=-0.0584090180117 -0.0871141177902 0.0330432309241 rpy=1.64075108736 0.0171079670332 -1.54271074297
