Commit message: 修改支持isaacsim仿真机械臂

File: src/rm_engineering_moveit_config/config/rm_engineering_robot.ros2_control.xacro (robot description, xacro)
@@ -1,15 +1,30 @@
 <?xml version="1.0"?>
 <robot xmlns:xacro="http://www.ros.org/wiki/xacro">
-    <xacro:macro name="rm_engineering_robot_ros2_control" params="name initial_positions_file">
+    <xacro:macro name="rm_engineering_robot_ros2_control" params="name initial_positions_file hardware_type:=real" >
         <xacro:property name="initial_positions" value="${load_yaml(initial_positions_file)['initial_positions']}"/>
+<!--        <xacro:arg name="hardware_type" default="real"/>-->
         <ros2_control name="${name}" type="system">
             <hardware>
                 <!-- By default, set up controllers for simulation. This won't work on real hardware -->
-                <plugin>engineering_hardware/EngineeringSystem</plugin>
-                <param name="device_name">/dev/ttyACM0</param>
-                <param name="baud_rate">115200</param>
-                <param name="fc_string">none</param>
-                <param name="pt_string">none</param>
-                <param name="sb_string">1</param>
+<!--                <plugin>engineering_hardware/EngineeringSystem</plugin>-->
+<!--                <param name="device_name">/dev/ttyACM0</param>-->
+<!--                <param name="baud_rate">115200</param>-->
+<!--                <param name="fc_string">none</param>-->
+<!--                <param name="pt_string">none</param>-->
+<!--                <param name="sb_string">1</param>-->
+                <xacro:if value="${hardware_type == 'real'}">
+                    <plugin>engineering_hardware/EngineeringSystem</plugin>
+                    <param name="device_name">/dev/ttyACM0</param>
+                    <param name="baud_rate">115200</param>
+                    <param name="fc_string">none</param>
+                    <param name="pt_string">none</param>
+                    <param name="sb_string">1</param>
+                </xacro:if>
+                <!-- Isaac Sim 接口 -->
+                <xacro:if value="${hardware_type == 'isaac'}">
+                    <plugin>topic_based_ros2_control/TopicBasedSystem</plugin>
+                    <param name="joint_commands_topic">/isaac_joint_commands</param>
+                    <param name="joint_states_topic">/isaac_joint_states</param>
+                </xacro:if>
             </hardware>
             <joint name="joint0">

File: src/rm_engineering_moveit_config/config/rm_engineering_robot.urdf.xacro (robot description, xacro)
@@ -1,4 +1,6 @@
 <?xml version="1.0"?>
 <robot xmlns:xacro="http://www.ros.org/wiki/xacro" name="rm_engineering_robot">
+    <!--使用实车硬件接口还是isaac接口-->
+    <xacro:arg name="hardware_type" default="real"/>
     <xacro:arg name="initial_positions_file" default="initial_positions.yaml" />
     <!-- Import rm_engineering_robot urdf file -->
@@ -6,4 +8,4 @@
     <!-- Import control_xacro -->
     <xacro:include filename="rm_engineering_robot.ros2_control.xacro" />
-    <xacro:rm_engineering_robot_ros2_control name="FakeSystem" initial_positions_file="$(arg initial_positions_file)"/>
+    <xacro:rm_engineering_robot_ros2_control name="FakeSystem" initial_positions_file="$(arg initial_positions_file)" hardware_type="$(arg hardware_type)"/>
 </robot>

File: src/rm_engineering_robot_description/urdf/rm_engineering_robot.urdf (robot description, URDF)
Before this commit: robot rm_engineering_robot, 9 links, 8 joints
Links:
- link base_link: geometry collision box size=0.4 0.4 0.6; visual mesh filename=package://rm_engineering_robot_description/meshes/base_link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
